File: Hardware/KiCAD_Project_Files/Arduino_LCD_Experimenter_Shield.sch (KiCad schematic (older format))
At the start: 51 parts

Commit message: Created new decals and footprints with 3D models
Parts:
- removed D? (x3): LED, symbol LED
- removed D? (x2): DIODE_SCHOTTKY, symbol DIODE_SCHOTTKY
- removed LS?: PS1240P02BT, symbol PIEZO_TRANSDUCER
- removed P?: HEADER_2X3, symbol HEADER_2X3
- removed P? (x2): HEADER_1X8, symbol HEADER_1X8
- removed P?: HEADER_1X6, symbol HEADER_1X6
- removed P?: HEADER_1X10, symbol HEADER_1X10
- removed SW? (x6): PTS810 SJM, symbol FSMSM
- removed TP?: 5015, symbol 5015
- removed U?: MCP23008E/SO, symbol MCP23008E/SO
- removed X?: 32.768kHz, symbol CRYSTAL
- added D4: BAV70L, symbol BAV70L
- added DS1, DS2, DS3: YEL, symbol LED
- added DS4: HDG1602P-1, symbol HDG1602P-1
- added LS1: PS1240P02BT, symbol PS1240P02BT
- added P1: 1X10 HEADER, symbol HEADER_M_2.54MM_1R10P_ST_AU_PTH
- added P2, P4: 1X8 HEADER, symbol HEADER_M_2.54MM_1R8P_ST_AU_PTH
- added P3: 1X6 HEADER, symbol HEADER_M_2.54MM_1R6P_ST_AU_PTH
- added P5: 2X3 HEADER, symbol HEADER_M_2.54MM_2R6P_ST_AU_PTH
- added SW1, SW2, SW3, SW4, SW5, SW6: PTS810, symbol PTS810
- added U1: MCP23008E/SS, symbol MCP23008E/SS
- added W1: WIRE_PAD_26AWG, symbol WIRE_PAD_26AWG
- added X1: 32.768k, symbol AB26TRQ
- BT1: renamed from BT?; value BATTERY_3PIN -> BK-912 (2032)
- C2, C3: renamed from C?; value CAP -> 8pF
- R1, R2, R3: renamed from R?; value RES_SMALL -> 270
- gave numbers to parts that had none: 25
Connections:
- net labels added: RW
- net labels removed: 5V, R/W
- wire segments 230 -> 211
- no-connect marks 8 -> 1
Other:
- note added: "BAT-HLD-012-SMT (1216)"
- note removed: "TODO:\n - Check crystal connection/components for RTC"
